Commit message: Added simple continous command example

File: joint_controller_ros2_control/test/urdf/core/single_joint.urdf.xacro (robot description, xacro)
@@ -46,5 +46,5 @@
             </geometry>
             <material name="">
-                <color rgba="0.0 1.0 0.0 1.0"/>
+                <color rgba="0.0 0.0 1.0 1.0"/>
             </material>
         </visual>

File: joint_controller_ros2_control/test/urdf/single_joint_test.urdf.xacro (robot description, xacro)
@@ -3,8 +3,8 @@
     <xacro:property name="PI" value="3.141592"/>
     <xacro:property name="rotor_inertia" value="1.0"/>
-    <xacro:property name="rotor_position_max" value="${PI}"/>
-    <xacro:property name="rotor_position_min" value="${-PI}"/>
-    <xacro:property name="rotor_velocity_max" value="10.0"/>
-    <xacro:property name="rotor_effort_max" value="10.0"/>
+    <xacro:property name="rotor_position_max" value="${10 * PI}"/>
+    <xacro:property name="rotor_position_min" value="${-10 * PI}"/>
+    <xacro:property name="rotor_velocity_max" value="50.0"/>
+    <xacro:property name="rotor_effort_max" value="50.0"/>
     <link name="world"/>
     <!-- Single joint macro -->
